Commit message: added sine generator and README

File: config/xacro/imu.urdf.xacro (robot description, xacro)
@@ -6,5 +6,5 @@
       <origin xyz="-2.08 0.72 4.22" rpy="0 0 0" />
       <geometry>
-        <mesh filename="package://tracking_master/config/meshes/IMUBox.stl" scale="0.005 0.005 0.005"/>
+        <mesh filename="package://odor_tracker/config/meshes/IMUBox.stl" scale="0.005 0.005 0.005"/>
       </geometry>
     </visual>

File: config/xacro/main.urdf.xacro (robot description, xacro)
@@ -1,5 +1,5 @@
 <?xml version="1.0"?>
 <robot name="dronemockup" xmlns:xacro="http://ros.org/wiki/xacro">
-     <xacro:include filename="$(find tracking_master)/config/xacro/imu.urdf.xacro" />
+     <xacro:include filename="$(find odor_tracker)/config/xacro/imu.urdf.xacro" />
   <xacro:arg name="robot_namespace" default="/" />
   <xacro:property name="M_PI" value="3.14159"/>
@@ -9,5 +9,5 @@
       <origin xyz="0 0 0" rpy="0 -${M_PI/2} 0" />
       <geometry>
-        <mesh filename="package://tracking_master/config/meshes/frame.STL" scale="0.005 0.005 0.005"/>
+        <mesh filename="package://odor_tracker/config/meshes/frame.STL" scale="0.005 0.005 0.005"/>
       </geometry>
     </visual>
@@ -18,5 +18,5 @@
       <origin xyz="-2.14 0.72 4.15" rpy="${M_PI/2} 0 -${M_PI/2}" />
       <geometry>
-        <mesh filename="package://tracking_master/config/meshes/T265.stl" scale="0.005 0.005 0.005"/>
+        <mesh filename="package://odor_tracker/config/meshes/T265.stl" scale="0.005 0.005 0.005"/>
       </geometry>
     </visual>
@@ -32,5 +32,5 @@
       <origin xyz="-2.14 0.72 4.15" rpy="${M_PI/2} 0 -${M_PI/2}" />
       <geometry>
-        <mesh filename="package://tracking_master/config/meshes/T265.stl" scale="0.005 0.005 0.005"/>
+        <mesh filename="package://odor_tracker/config/meshes/T265.stl" scale="0.005 0.005 0.005"/>
       </geometry>
     </visual>
@@ -46,5 +46,5 @@
       <origin xyz="-2.08 -0.7 4.28" rpy="${M_PI/2} ${M_PI/2} 0" />
       <geometry>
-        <mesh filename="package://tracking_master/config/meshes/basler.stl" scale="0.004 0.004 0.004"/>
+        <mesh filename="package://odor_tracker/config/meshes/basler.stl" scale="0.004 0.004 0.004"/>
       </geometry>
     </visual>
@@ -63,5 +63,5 @@
       <origin xyz="-2.08 -0.03 4.22" rpy="0 0 0" />
       <geometry>
-        <mesh filename="package://tracking_master/config/meshes/ballscrew.stl" scale="0.004 0.004 0.004"/>
+        <mesh filename="package://odor_tracker/config/meshes/ballscrew.stl" scale="0.004 0.004 0.004"/>
       </geometry>
     </visual>
@@ -77,5 +77,5 @@
       <origin xyz="-2.15 -0.1 4.6" rpy="0 0 0" />
       <geometry>
-        <mesh filename="package://tracking_master/config/meshes/trisonicamount.stl" scale="0.004 0.004 0.004"/>
+        <mesh filename="package://odor_tracker/config/meshes/trisonicamount.stl" scale="0.004 0.004 0.004"/>
       </geometry>
     </visual>
@@ -91,5 +91,5 @@
       <origin xyz="-1.2 -0.03 4.22" rpy="0 0 0" />
       <geometry>
-        <mesh filename="package://tracking_master/config/meshes/IMUBox.stl" scale="0.004 0.004 0.004"/>
+        <mesh filename="package://odor_tracker/config/meshes/IMUBox.stl" scale="0.004 0.004 0.004"/>
       </geometry>
     </visual>

File: config/xacro/t265.urdf.xacro (robot description, xacro)
@@ -6,5 +6,5 @@
       <origin xyz="0 0 0" rpy="0 0 0" />
       <geometry>
-        <mesh filename="package://tracking_master/config/meshes/T265.stl" />
+        <mesh filename="package://odor_tracker/config/meshes/T265.stl" />
       </geometry>
     </visual>
